File: RAMPS_1.6.2.brd (EAGLE design)
At the start: 130 x 60 mm, 101 parts, among them Q1 STP55NF06L, Q2 STP55NF06L, Q3 STP55NF06L

Commit message: changed package to 1206 on R and C
Parts:
- C11, C13, C15: device rcl:C0805 -> rcl:C1206
- C2: device resistor:C0805 -> resistor:C1206
- LED1, LED10, LEDD8, LEDD9: device led:CHIP-LED0805 -> led:CHIPLED_1206
- R1, R10, R11, R12, R16, R17, R2, R23, R24, R25, R3, R4, R5, R6, R7, R8, R9: device adafruit:R0805 -> adafruit:R1206
- R13, R15: device resistor:R0805 -> resistor:R1206
- R14: device resistor:M0805 -> resistor:R1206
- R18, R19, R20, R26, R27, R28, R29, R30, R31, R32, R33, R34, R35, R36, R37: device resistor:M1206 -> resistor:R1206
- moved R28 0.90 mm to (105.0, 67.2)
Routing:
- net +12V: track 240.6 -> 382.0 mm
- net GND: track 273.4 -> 285.8 mm
- net N$50: track 1.79 -> 0.67 mm
- net N$1: track 34.5 -> 33.4 mm
- net HEAT3: track 32.4 -> 33.2 mm
- net N$7: track 26.1 -> 25.6 mm

Commit message: changed few componments for Order
Parts:
- removed S2: reset, switch:SKHMPXE010
- added U$2: RS-TASTER, My lib:RS-SWITCH
- F1, F2: value SMD-AUTOMOTIVE-FUSE -> SMD-AUTOMOTIVE-FUSEREICHELTVARIANTE; device My lib:BLADEFUSE -> My lib:RS-SMDFUSE
- moved R23 10.7 mm to (19.6, 54.0), turned to 180 degrees
- moved F1 9.44 mm to (14.9, 35.3)
- moved F2 7.24 mm to (12.8, 22.0)
- moved C2 1.42 mm to (27.2, 36.2)
- moved LEDD8 1.27 mm to (10.1, 55.8)
- moved R25 1.27 mm to (10.1, 68.9)
- moved D2 0.90 mm to (19.8, 33.7)
- moved R6 0.78 mm to (91.8, 42.1), turned to 90 degrees
- moved C15 0.64 mm to (103.5, 43.8)
- moved R12 0.64 mm to (77.5, 14.9)
- moved R16 0.64 mm to (89.9, 65.5)
- moved C13 0.63 mm to (103.4, 33.0)
Connections:
- net +12V: now also F1.P$5, F1.P$6, F1.P$7, F1.P$8; no longer F1.2, F1.2@2
- net +24V: now also F2.P$5, F2.P$6, F2.P$7, F2.P$8; no longer F2.2, F2.2@2
- net GND: now also U$2.P$1, U$2.P$2; no longer S2.1, S2.2
- net N$53: now also F2.P$1, F2.P$2, F2.P$3, F2.P$4; no longer F2.1, F2.1@1
- net N$54: now also F1.P$1, F1.P$2, F1.P$3, F1.P$4; no longer F1.1, F1.1@1
- net RESET: now also U$2.P$3, U$2.P$4; no longer S2.3
Routing:
- net N$53: track 10.8 -> 38.1 mm
- net +12V: track 382.0 -> 406.8 mm
- net +24V: track 94.1 -> 111.6 mm
- net GND: track 285.8 -> 301.6 mm
- net RESET: track 9.39 -> 19.6 mm
- net N$32: track 2.52 -> 8.63 mm
- net N$1: track 33.4 -> 28.3 mm
- net N$54: track 13.9 -> 19.1 mm
- net VCC: track 112.1 -> 115.8 mm
- net E0-STEP: track 37.4 -> 38.9 mm
- net N$50: track 0.67 -> 1.94 mm
- net X-DIR: track 103.2 -> 104.3 mm
- net HEAT2: track 21.3 -> 22.3 mm
- net N$51: track 17.6 -> 16.6 mm
- net N$42: track 17.7 -> 16.8 mm
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