File: RAMPS_1.6.2.sch (EAGLE design)
At the start: 101 parts, among them Q1 STP55NF06L, Q2 STP55NF06L, Q3 STP55NF06L

Commit message: changed package to 1206 on R and C
Parts:
- C11, C13, C15: device rcl:C-EUC0805 -> rcl:C-EUC1206
- C2: device resistor:C-EUC0805 -> resistor:C-EUC1206
- LED1, LED10, LEDD8, LEDD9: device led:LEDCHIP-LED0805 -> led:LEDCHIPLED_1206
- R1, R10, R11, R12, R16, R17, R2, R23, R24, R25, R3, R4, R5, R6, R7, R8, R9: device adafruit:R-US_R0805 -> adafruit:R-US_R1206
- R13, R15: device resistor:R-US_R0805 -> resistor:R-US_R1206
- R14: device resistor:R-US_M0805 -> resistor:R-US_R1206
- R18, R19, R20, R26, R27, R28, R29, R30, R31, R32, R33, R34, R35, R36, R37: device resistor:R-US_M1206 -> resistor:R-US_R1206

Commit message: Add files via upload
Parts:
- removed S2: reset, switch:SKHMPWE010
- added U$2: RS-TASTER, My lib:RS-TASTER
- F1, F2: value SMD-AUTOMOTIVE-FUSE -> SMD-AUTOMOTIVE-FUSEREICHELTVARIANTE; device My lib:SMD-AUTOMOTIVE-FUSE -> My lib:SMD-AUTOMOTIVE-FUSEREICHELTVARIANTE
Connections:
- net GND: now also U$2.P$1, U$2.P$2; no longer S2.1.1, S2.1.2
- net RESET: now also U$2.P$3, U$2.P$4; no longer S2.2.1
